Commit message: xyz linear carriage

File: urdf/06-flexible.urdf (robot description, URDF)
Before this commit: robot cart, 3 links, 2 joints
Links:
- removed link cart
- removed link slideBar
- added link follower_x, mass 1; visual box size=0.01 0.01 0.01
- added link follower_y, mass 1; visual box size=0.01 0.01 0.01
- added link follower_z, mass 1; visual box size=0.01 0.01 0.01
Joints:
- removed joint slider_to_cart
- removed joint world_to_base
- added joint follower_x_to_follower_y: type prismatic, parent follower_x, child follower_y, origin xyz=0.0 0.0 0.0, axis 0 1 0, limit lower=-9999 upper=9999 effort=1000.0 velocity=9999
- added joint follower_y_to_follower_z: type prismatic, parent follower_y, child follower_z, origin xyz=0.0 0.0 0.0, axis 0 0 1, limit lower=-9999 upper=9999 effort=1000.0 velocity=9999
- added joint world_to_follower_x: type prismatic, parent world, child follower_x, origin xyz=0.0 0.0 0.0, axis 1 0 0, limit lower=-9999 upper=9999 effort=1000.0 velocity=9999
